Commit message: Controller Finish

File: ROS_ws/src/arduinobot_description/urdf/arduinobot_ros2_control.xacro (robot description, xacro)
@@ -27,4 +27,20 @@
             <state_interface name="position"/>
         </joint>
+        <!-- <joint name="joint_4">
+            <command_interface name="position">
+                <param name="min">-${PI/2}</param>
+                <param name="max">0.0</param>
+            </command_interface>
+            <state_interface name="position"/>
+        </joint>
+        <joint name="joint_5">
+            <param name="mimic">joint_4</param>
+            <param name="multiplier">-1</param>
+            <command_interface name="position">
+                <param name="min">0.0</param>
+                <param name="max">${PI/2}</param>
+            </command_interface>
+            <state_interface name="position"/>
+        </joint> -->
     </ros2_control>
 </robot>
