Commit message: Edited Arduinobot Description for BRACCIO bot model
- Note: renamed certain folders and files to clarify it's the braccio bot (branch)
- Replaced meshes
- Wrote braccio.urdf.xacro (original braccio urdf missing components/bugs)
- Edited ros2_control.xacro, controller.yaml, and etc., files

File: ROS_ws/src/arduinobot_braccio_description/urdf/braccio_ros2_control.xacro (robot description, xacro)
@@ -6,5 +6,5 @@
             <plugin>gazebo_ros2_control/GazeboSystem</plugin>
         </hardware>
-        <joint name="joint_1">
+        <joint name="base">
             <command_interface name="position">
                 <param name="min">-${PI/2}</param>
@@ -13,5 +13,5 @@
             <state_interface name="position"/>
         </joint>
-        <joint name="joint_2">
+        <joint name="shoulder">
             <command_interface name="position">
                 <param name="min">-${PI/2}</param>
@@ -20,5 +20,5 @@
             <state_interface name="position"/>
         </joint>
-        <joint name="joint_3">
+        <joint name="elbow">
             <command_interface name="position">
                 <param name="min">-${PI/2}</param>
@@ -27,20 +27,25 @@
             <state_interface name="position"/>
         </joint>
-        <!-- <joint name="joint_4">
+        <joint name="wrist_pitch">
             <command_interface name="position">
                 <param name="min">-${PI/2}</param>
-                <param name="max">0.0</param>
+                <param name="max">${PI/2}</param>
             </command_interface>
             <state_interface name="position"/>
         </joint>
-        <joint name="joint_5">
-            <param name="mimic">joint_4</param>
-            <param name="multiplier">-1</param>
+        <joint name="wrist_roll">
             <command_interface name="position">
-                <param name="min">0.0</param>
+                <param name="min">-${PI/2}</param>
                 <param name="max">${PI/2}</param>
             </command_interface>
             <state_interface name="position"/>
-        </joint> -->
+        </joint>
+        <joint name="gripper_movable">
+            <command_interface name="position">
+                <param name="min">0.0</param>
+                <param name="max">${PI/4}</param>
+            </command_interface>
+            <state_interface name="position"/>
+        </joint>
     </ros2_control>
 </robot>

Commit message: Finished & Working Launch MoveIt!
- Added initial values to ros2_control.xacro file as new param
- (may have made initial_position.yaml redundant but matched intial values there just in case)
- Matched initial values in srdf for consistency (other values didn't seem to change anything)
- Fixed bug in moveitcontrollers.yaml (type had to be camel case not snake case)
- Saved rviz working config as moveit.rviz for convenience

File: ROS_ws/src/arduinobot_braccio_description/urdf/braccio_ros2_control.xacro (robot description, xacro)
@@ -1,5 +1,5 @@
 <?xml version="1.0"?>
 <robot xmlns:xacro="https://www.ros.org/wiki/xacro" name="arduinobot">
-    <xacro:property name="PI" value="3.14159"/>
+    <xacro:property name="PI" value="3.141592653589793"/>
     <ros2_control name="RobotSystem" type="system">
         <hardware>
@@ -8,43 +8,55 @@
         <joint name="base">
             <command_interface name="position">
-                <param name="min">-${PI/2}</param>
-                <param name="max">${PI/2}</param>
+                <param name="min">0</param>
+                <param name="max">${PI}</param>
             </command_interface>
-            <state_interface name="position"/>
+            <state_interface name="position">
+                <param name="initial_value">0</param>
+            </state_interface>
         </joint>
         <joint name="shoulder">
             <command_interface name="position">
-                <param name="min">-${PI/2}</param>
-                <param name="max">${PI/2}</param>
+                <param name="min">0.2617993877991494</param>
+                <param name="max">2.8797932657906435</param>
             </command_interface>
-            <state_interface name="position"/>
+            <state_interface name="position">
+                <param name="initial_value">${PI/2}</param>
+            </state_interface>
         </joint>
         <joint name="elbow">
             <command_interface name="position">
-                <param name="min">-${PI/2}</param>
-                <param name="max">${PI/2}</param>
+                <param name="min">0</param>
+                <param name="max">${PI}</param>
             </command_interface>
-            <state_interface name="position"/>
+            <state_interface name="position">
+                <param name="initial_value">${PI/2}</param>
+            </state_interface>
         </joint>
         <joint name="wrist_pitch">
             <command_interface name="position">
-                <param name="min">-${PI/2}</param>
-                <param name="max">${PI/2}</param>
+                <param name="min">0</param>
+                <param name="max">${PI}</param>
             </command_interface>
-            <state_interface name="position"/>
+            <state_interface name="position">
+                <param name="initial_value">${PI/2}</param>
+            </state_interface>
         </joint>
         <joint name="wrist_roll">
             <command_interface name="position">
-                <param name="min">-${PI/2}</param>
-                <param name="max">${PI/2}</param>
+                <param name="min">0</param>
+                <param name="max">${PI}</param>
             </command_interface>
-            <state_interface name="position"/>
+            <state_interface name="position">
+                <param name="initial_value">${PI/2}</param>
+            </state_interface>
         </joint>
         <joint name="gripper_movable">
             <command_interface name="position">
-                <param name="min">0.0</param>
-                <param name="max">${PI/4}</param>
+                <param name="min">0.17453292519943295</param>
+                <param name="max">1.2740903539558606</param>
             </command_interface>
-            <state_interface name="position"/>
+            <state_interface name="position">
+                <param name="initial_value">0.724</param>
+            </state_interface>
         </joint>
     </ros2_control>
