Commit message: Launch MoveIt Progress
- Fixed Bugs
--> e.g. fixed incorrectly named file
--> e.g. edited moveit config files for braccio urdf
- Removed base_link in urdf
--> was causing Gazebo issue, now fixed!!
--> also fixed small bug in macro
- PROBLEM
--> launching controller.launch.py now doesn't work
--> should make bot move to intial, makes it contort into out of range

File: ROS_ws/src/arduinobot_braccio_description/urdf/braccio.urdf.xacro (robot description, xacro)
@@ -1,5 +1,5 @@
 <?xml version="1.0"?>
 <robot xmlns:xacro="https://www.ros.org/wiki/xacro" name="arduinobot">
-  <!-- <xacro:include filename="$(find arduinobot_braccio_description)/urdf/arduinobot_gazebo.xacro"/> -->
+  <xacro:include filename="$(find arduinobot_braccio_description)/urdf/arduinobot_gazebo.xacro"/>
   <xacro:include filename="$(find arduinobot_braccio_description)/urdf/braccio_ros2_control.xacro"/>
   <xacro:property name="PI" value="3.14159"/>
@@ -20,5 +20,5 @@
           </plugin>
           <actuator name="motor_${name}" role="actuator1"/>
-          <joint name="joint_${name}" role="joint1">
+          <joint name="${name}" role="joint1">
               <mechanical_reduction>
                   1.0
@@ -37,21 +37,4 @@
   </material>
   <link name="world"/>
-  <link name="base_link">
-    <xacro:default_inertial mass="1.0"/>
-    <visual>
-      <geometry>
-        <box size="0.15 0.15 .05"/>
-      </geometry>
-      <material name="gray"/>
-      <origin rpy="0 0 0" xyz="0 0 -0.025"/>
-    </visual>
-    <collision>
-      <geometry>
-        <box size="0.15 0.15 .05"/>
-      </geometry>
-      <material name="gray"/>
-      <origin rpy="0 0 0" xyz="0 0 -0.025"/>
-    </collision>
-  </link>
   <link name="link1">
     <xacro:default_inertial mass="1.0"/>
@@ -188,15 +171,9 @@
     </collision>
   </link>
-  <joint name="worldBaseJoint" type="fixed">
-    <axis xyz="0 0 0"/>
-    <origin rpy="0 0 0" xyz="0 0 0"/>
-    <parent link="world"/>
-    <child link="base_link"/>
-  </joint>
   <joint name="base" type="revolute">
     <axis xyz="0 0 -1"/>
     <limit effort="1000.0" lower="0.0" upper="3.141592653589793" velocity="4.0"/>
     <origin rpy="0 0 0" xyz="0 0 0"/>
-    <parent link="base_link"/>
+    <parent link="world"/>
     <child link="link1"/>
   </joint>

Commit message: Replaced Braccio Model and adjusted files accordingly

File: ROS_ws/src/arduinobot_braccio_description/urdf/braccio.urdf.xacro (robot description, xacro)
@@ -38,135 +38,118 @@
   <link name="world"/>
   <link name="link1">
+    <xacro:default_inertial mass="2.0"/>
+    <visual>
+      <geometry>
+        <mesh filename="package://arduinobot_braccio_description/meshes/base.stl" scale="0.001 0.001 0.001" />
+      </geometry>
+      <material name="orange"/>
+    </visual>
+    <collision>
+      <geometry>
+        <mesh filename="package://arduinobot_braccio_description/meshes/base.stl" scale="0.001 0.001 0.001" />
+      </geometry>
+      <material name="orange"/>
+    </collision>
+  </link>
+  <link name="link2">
+    <xacro:default_inertial mass="0.1"/>
+    <visual>
+      <geometry>
+        <mesh filename="package://arduinobot_braccio_description/meshes/shoulder.stl" scale="0.001 0.001 0.001" />
+      </geometry>
+      <material name="orange"/>
+      <origin rpy="0 0 0" xyz="-0.0045 0.0055 -0.026" />
+    </visual>
+    <collision>
+      <geometry>
+        <mesh filename="package://arduinobot_braccio_description/meshes/shoulder.stl" scale="0.001 0.001 0.001" />
+      </geometry>
+      <material name="orange"/>
+      <origin rpy="0 0 0" xyz="-0.0045 0.0055 -0.026" />
+    </collision>
+  </link>
+  <link name="link3">
+    <xacro:default_inertial mass="0.1"/>
+    <visual>
+      <geometry>
+        <mesh filename="package://arduinobot_braccio_description/meshes/elbow.stl" scale="0.001 0.001 0.001" />
+      </geometry>
+      <material name="orange"/>
+      <origin rpy="0 0 0" xyz="-0.0045 0.005 -0.025" />
+    </visual>
+    <collision>
+      <geometry>
+        <mesh filename="package://arduinobot_braccio_description/meshes/elbow.stl" scale="0.001 0.001 0.001" />
+      </geometry>
+      <material name="orange"/>
+      <origin rpy="0 0 0" xyz="-0.0045 0.005 -0.025" />
+    </collision>
+  </link>
+  <link name="link4">
+    <xacro:default_inertial mass="0.1"/>
+    <visual>
+      <geometry>
+        <mesh filename="package://arduinobot_braccio_description/meshes/wrist_pitch.stl" scale="0.001 0.001 0.001" />
+      </geometry>
+      <material name="orange"/>
+      <origin rpy="0 0 0" xyz="0.003 -0.0004 -0.024" />
+    </visual>
+    <collision>
+      <geometry>
+        <mesh filename="package://arduinobot_braccio_description/meshes/wrist_pitch.stl" scale="0.001 0.001 0.001" />
+      </geometry>
+      <material name="orange"/>
+      <origin rpy="0 0 0" xyz="0.003 -0.0004 -0.024" />
+    </collision>
+  </link>
+  <link name="link5">
+    <xacro:default_inertial mass="0.1"/>
+    <visual>
+      <geometry>
+        <mesh filename="package://arduinobot_braccio_description/meshes/wrist_roll.stl" scale="0.001 0.001 0.001" />
+      </geometry>
+      <material name="white"/>
+      <origin rpy="0 0 0" xyz="0.006 0 0.0" />
+    </visual>
+    <collision>
+      <geometry>
+        <mesh filename="package://arduinobot_braccio_description/meshes/wrist_roll.stl" scale="0.001 0.001 0.001" />
+      </geometry>
+      <material name="white"/>
+      <origin rpy="0 0 0" xyz="0.006 0 0.0" />
+    </collision>
+  </link>
+  <link name="gripper_right">
     <xacro:default_inertial mass="1.0"/>
     <visual>
       <geometry>
-        <mesh filename="package://arduinobot_braccio_description/meshes/base.stl"/>
-      </geometry>
-      <material name="orange"/>
-    </visual>
-    <collision>
-      <geometry>
-        <mesh filename="package://arduinobot_braccio_description/meshes/base.stl"/>
-      </geometry>
-      <material name="orange"/>
-    </collision>
-  </link>
-  <link name="link2">
+        <mesh filename="package://arduinobot_braccio_description/meshes/right_gripper.stl" scale="0.001 0.001 0.001" />
+      </geometry>
+      <material name="white"/>
+      <origin rpy="0 1.5708 0" xyz="0 -0.012 0.010" />
+    </visual>
+    <collision>
+      <geometry>
+        <mesh filename="package://arduinobot_braccio_description/meshes/right_gripper.stl" scale="0.001 0.001 0.001" />
+      </geometry>
+      <material name="white"/>
+      <origin rpy="0 1.5708 0" xyz="0 -0.012 0.010" />
+    </collision>
+  </link>
+  <link name="gripper_left">
     <xacro:default_inertial mass="1.0"/>
     <visual>
       <geometry>
-        <mesh filename="package://arduinobot_braccio_description/meshes/shoulder.stl"/>
-      </geometry>
-      <material name="orange"/>
-      <origin rpy="0 0 0" xyz="0 0 -0.0505"/>
-    </visual>
-    <collision>
-      <geometry>
-        <mesh filename="package://arduinobot_braccio_description/meshes/shoulder.stl"/>
-      </geometry>
-      <material name="orange"/>
-      <origin rpy="0 0 0" xyz="0 0 -0.0505"/>
-    </collision>
-  </link>
-  <link name="link3">
-    <xacro:default_inertial mass="1.0"/>
-    <visual>
-      <geometry>
-        <mesh filename="package://arduinobot_braccio_description/meshes/elbow.stl"/>
-      </geometry>
-      <material name="orange"/>
-      <origin rpy="0 0 0" xyz="0 0 -0.1705"/>
-    </visual>
-    <collision>
-      <geometry>
-        <mesh filename="package://arduinobot_braccio_description/meshes/elbow.stl"/>
-      </geometry>
-      <material name="orange"/>
-      <origin rpy="0 0 0" xyz="0 0 -0.1705"/>
-    </collision>
-  </link>
-  <link name="link4">
-    <xacro:default_inertial mass="1.0"/>
-    <visual>
-      <geometry>
-        <mesh filename="package://arduinobot_braccio_description/meshes/wrist_pitch.stl"/>
-      </geometry>
-      <material name="orange"/>
-      <origin rpy="0 0 0" xyz="0 0 -0.2905"/>
-    </visual>
-    <collision>
-      <geometry>
-        <mesh filename="package://arduinobot_braccio_description/meshes/wrist_pitch.stl"/>
-      </geometry>
-      <material name="orange"/>
-      <origin rpy="0 0 0" xyz="0 0 -0.2905"/>
-    </collision>
-  </link>
-  <link name="link5">
-    <xacro:default_inertial mass="1.0"/>
-    <visual>
-      <geometry>
-        <mesh filename="package://arduinobot_braccio_description/meshes/wrist_roll.stl"/>
-      </geometry>
-      <material name="white"/>
-      <origin rpy="0 0 0" xyz="0 0 -0.3505"/>
-    </visual>
-    <collision>
-      <geometry>
-        <mesh filename="package://arduinobot_braccio_description/meshes/wrist_roll.stl"/>
-      </geometry>
-      <material name="white"/>
-      <origin rpy="0 0 0" xyz="0 0 -0.3505"/>
-    </collision>
-  </link>
-  <link name="gripper_base">
-    <xacro:default_inertial mass="1.0"/>
-    <visual>
-      <geometry>
-        <mesh filename="package://arduinobot_braccio_description/meshes/gripper_base.stl"/>
-      </geometry>
-      <material name="white"/>
-      <origin rpy="0 0 0" xyz="0 0 -0.357"/>
-    </visual>
-    <collision>
-      <geometry>
-        <mesh filename="package://arduinobot_braccio_description/meshes/gripper_base.stl"/>
-      </geometry>
-      <material name="white"/>
-      <origin rpy="0 0 0" xyz="0 0 -0.357"/>
-    </collision>
-  </link>
-  <link name="gripper_fix">
-    <xacro:default_inertial mass="1.0"/>
-    <visual>
-      <geometry>
-        <mesh filename="package://arduinobot_braccio_description/meshes/gripper_fix.stl"/>
-      </geometry>
-      <material name="white"/>
-      <origin rpy="0 0 0" xyz="0 0 -0.36399"/>
-    </visual>
-    <collision>
-      <geometry>
-        <mesh filename="package://arduinobot_braccio_description/meshes/gripper_fix.stl"/>
-      </geometry>
-      <material name="white"/>
-      <origin rpy="0 0 0" xyz="0 0 -0.36399"/>
-    </collision>
-  </link>
-  <link name="gripper_movable_link">
-    <xacro:default_inertial mass="1.0"/>
-    <visual>
-      <geometry>
-        <mesh filename="package://arduinobot_braccio_description/meshes/gripper_movable_link.stl"/>
-      </geometry>
-      <material name="white"/>
-      <origin rpy="0 0 0" xyz="-0.01559 0 -0.36399"/>
-    </visual>
-    <collision>
-      <geometry>
-        <mesh filename="package://arduinobot_braccio_description/meshes/gripper_movable_link.stl"/>
-      </geometry>
-      <material name="white"/>
-      <origin rpy="0 0 0" xyz="-0.01559 0 -0.36399"/>
+        <mesh filename="package://arduinobot_braccio_description/meshes/left_gripper.stl" scale="0.001 0.001 0.001" />
+      </geometry>
+      <material name="white"/>
+      <origin rpy="0 1.5708 0" xyz="0 -0.012 0" />
+    </visual>
+    <collision>
+      <geometry>
+        <mesh filename="package://arduinobot_braccio_description/meshes/left_gripper.stl" scale="0.001 0.001 0.001" />
+      </geometry>
+      <material name="white"/>
+      <origin rpy="0 1.5708 0" xyz="0 -0.012 0" />
     </collision>
   </link>
@@ -206,20 +189,18 @@
     <child link="link5"/>
   </joint>
-  <joint name="gripper_base" type="fixed">
-    <origin rpy="0 0 0" xyz="0 0.0 0.0065"/>
-    <parent link="link5"/>
-    <child link="gripper_base"/>
-  </joint>
-  <joint name="gripper_fix" type="fixed">
-    <origin rpy="0 0 0" xyz="0 0.0 0.007"/>
-    <parent link="gripper_base"/>
-    <child link="gripper_fix"/>
-  </joint>
-  <joint name="gripper_movable" type="revolute">
-    <axis xyz="0 -1 0"/>
-    <limit effort="1000.0" lower="0.17453292519943295" upper="1.2740903539558606" velocity="4.0"/>
-    <origin rpy="0 0 0" xyz="0.01559 0 0.007"/>
-    <parent link="gripper_base"/>
-    <child link="gripper_movable_link"/>
+  <joint name="gripper_joint" type="revolute">
+      <axis xyz="0 -1 0" />
+      <limit effort="1.0" lower="0.17453292519943295" upper="1.2740903539558606" velocity="1.0" />
+      <origin rpy="0 -0.2967 0" xyz="0.010 0 0.03" />
+      <parent link="link5" />
+      <child link="gripper_right" />
+  </joint>
+  <joint name="gripper_sub_joint" type="revolute">
+      <axis xyz="0 1 0" />
+      <limit effort="1.0" lower="0.17453292519943295" upper="1.2740903539558606" velocity="1.0" />
+      <origin rpy="0 3.4383 0" xyz="-0.010 0 0.03" />
+      <parent link="link5" />
+      <child link="gripper_left" />
+      <mimic joint="gripper_joint" multiplier="1"/>
   </joint>
   <xacro:default_transmission name="base"/>
@@ -228,4 +209,4 @@
   <xacro:default_transmission name="wrist_pitch"/>
   <xacro:default_transmission name="wrist_roll"/>
-  <xacro:default_transmission name="gripper_movable"/>
+  <xacro:default_transmission name="gripper_joint"/>
 </robot>

File: ROS_ws/src/arduinobot_braccio_description/urdf/braccio_ros2_control.xacro (robot description, xacro)
@@ -51,5 +51,5 @@
             </state_interface>
         </joint>
-        <joint name="gripper_movable">
+        <joint name="gripper_joint">
             <command_interface name="position">
                 <param name="min">0.17453292519943295</param>
@@ -60,4 +60,11 @@
             </state_interface>
         </joint>
+        <joint name="gripper_sub_joint">
+            <param name="mimic">gripper_joint</param>
+            <param name="multiplier">1</param>
+            <state_interface name="position">
+                <param name="initial_value">0.724</param>
+            </state_interface>
+        </joint>
     </ros2_control>
 </robot>

Commit message: ALMOST DONE!

File: ROS_ws/src/arduinobot_braccio_description/urdf/braccio.urdf.xacro (robot description, xacro)
@@ -1,4 +1,5 @@
 <?xml version="1.0"?>
 <robot xmlns:xacro="https://www.ros.org/wiki/xacro" name="arduinobot">
+  <xacro:arg name="is_sim" default="true"/>
   <xacro:include filename="$(find arduinobot_braccio_description)/urdf/arduinobot_gazebo.xacro"/>
   <xacro:include filename="$(find arduinobot_braccio_description)/urdf/braccio_ros2_control.xacro"/>
@@ -37,4 +38,9 @@
   </material>
   <link name="world"/>
+  <link name="random"/>
+  <joint name="gripper_sub_joint_mimic" type="fixed">
+    <parent link="world"/>
+    <child link="random"/>
+  </joint>
   <link name="link1">
     <xacro:default_inertial mass="2.0"/>

File: ROS_ws/src/arduinobot_braccio_description/urdf/braccio_ros2_control.xacro (robot description, xacro)
@@ -3,7 +3,22 @@
     <xacro:property name="PI" value="3.141592653589793"/>
     <ros2_control name="RobotSystem" type="system">
-        <hardware>
-            <plugin>gazebo_ros2_control/GazeboSystem</plugin>
-        </hardware>
+        <xacro:if value="${arg is_sim}">
+            <hardware>
+                <plugin>gazebo_ros2_control/GazeboSystem</plugin>
+            </hardware>
+            <joint name="gripper_sub_joint">
+                <param name="mimic">gripper_joint</param>
+                <param name="multiplier">1</param>
+                <state_interface name="position">
+                    <param name="initial_value">0.724</param>
+                </state_interface>
+            </joint>
+        </xacro:if>
+        <xacro:unless value="${arg is_sim}">
+            <hardware>
+                <plugin>arduinobot_controller/ArduinobotInterface</plugin>
+                <param name="port">/dev/ttyACM0</param>
+            </hardware>
+        </xacro:unless>
         <joint name="base">
             <command_interface name="position">
@@ -60,11 +75,4 @@
             </state_interface>
         </joint>
-        <joint name="gripper_sub_joint">
-            <param name="mimic">gripper_joint</param>
-            <param name="multiplier">1</param>
-            <state_interface name="position">
-                <param name="initial_value">0.724</param>
-            </state_interface>
-        </joint>
     </ros2_control>
 </robot>
